File: Hardware/glove_pcb/flex.kicad_sch (KiCad schematic)
At the start: 16 parts, among them J7 Potentiometers, J8 Potentiometers

Commit message: Made most of changes from meeting
Connections:
- net VCC_UC renamed +5V
Changed lines of the file:
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@@
   (junction (at 33.02 86.36) (diameter 0) (color 0 0 0 0)
   )
+  (junction (at 58.42 20.32) (diameter 0) (color 0 0 0 0)
+  )
   (junction (at 115.57 20.32) (diameter 0) (color 0 0 0 0)
   )
@@
   (junction (at 77.47 107.95) (diameter 0) (color 0 0 0 0)
   )
+  (junction (at 58.42 107.95) (diameter 0) (color 0 0 0 0)
+  )
   (junction (at 147.32 83.82) (diameter 0) (color 0 0 0 0)
   )
@@
     )
   )
-  (global_label "VCC_UC" (shape input) (at 58.42 20.32 180) (fields_autoplaced)
-    (effects (font (size 1.27 1.27)) (justify right))
-    (property "Intersheetrefs" "${INTERSHEET_REFS}" (at 48.2381 20.32 0)
-      (effects (font (size 1.27 1.27)) (justify right) hide)
-    )
-  )
   (global_label "POT_RING_3" (shape output) (at 115.57 88.9 0) (fields_autoplaced)
     (effects (font (size 1.27 1.27)) (justify left))
@@
     (property "Intersheetrefs" "${INTERSHEET_REFS}" (at 168.8713 44.45 0)
       (effects (font (size 1.27 1.27)) (justify left) hide)
-    )
-  )
-  (global_label "VCC_UC" (shape input) (at 58.42 107.95 180) (fields_autoplaced)
-    (effects (font (size 1.27 1.27)) (justify right))
-    (property "Intersheetrefs" "${INTERSHEET_REFS}" (at 48.2381 107.95 0)
-      (effects (font (size 1.27 1.27)) (justify right) hide)
     )
   )
@@
     )
   )
+  (symbol (lib_id "power:+5V") (at 58.42 107.95 180) (unit 1)
+    (in_bom yes) (on_board yes) (dnp no) (fields_autoplaced)
+    (property "Reference" "#PWR085" (at 58.42 104.14 0)
+      (effects (font (size 1.27 1.27)) hide)
+    )
+    (property "Value" "+5V" (at 58.42 113.03 0)
+      (effects (font (size 1.27 1.27)))
+    )
+    (property "Footprint" "" (at 58.42 107.95 0)
+      (effects (font (size 1.27 1.27)) hide)
+    )
+    (property "Datasheet" "" (at 58.42 107.95 0)
+      (effects (font (size 1.27 1.27)) hide)
+    )
+    (pin "1")
+    (instances
+      (project "glove_pcb"
+        (path "/747ff5f3-d342-40b0-8e4e-75b3a3063e75/bbbc9975-a050-48bd-8c18-11f2eff17087"
+          (reference "#PWR085") (unit 1)
+        )
+      )
+    )
+  )
   (symbol (lib_id "Device:R") (at 77.47 99.06 0) (unit 1)
     (in_bom yes) (on_board yes) (dnp no) (fields_autoplaced)
@@
         )
       )
+    )
+  )
+  (symbol (lib_id "power:+5V") (at 58.42 20.32 0) (unit 1)
+    (in_bom yes) (on_board yes) (dnp no) (fields_autoplaced)
+    (property "Reference" "#PWR084" (at 58.42 24.13 0)
+      (effects (font (size 1.27 1.27)) hide)
+    )
+    (property "Value" "+5V" (at 58.42 15.24 0)
+      (effects (font (size 1.27 1.27)))
+    )
+    (property "Footprint" "" (at 58.42 20.32 0)
+      (effects (font (size 1.27 1.27)) hide)
+    )
+    (property "Datasheet" "" (at 58.42 20.32 0)
+      (effects (font (size 1.27 1.27)) hide)
+    )
+    (pin "1")
+    (instances
+      (project "glove_pcb"
+        (path "/747ff5f3-d342-40b0-8e4e-75b3a3063e75/bbbc9975-a050-48bd-8c18-11f2eff17087"
+          (reference "#PWR084") (unit 1)
+        )
+      )
