File: Hardware/glove_pcb/flex.kicad_sch (KiCad schematic)
At the start: 20 parts, among them J5 302-R141, J6 302-R141, U10 BZA408B, U11 BZA408B, U8 BZA408B, U9 BZA408B

Commit message: Adjust placing based on size conflicts
Parts:
- J5, J6: footprint Connector_PinSocket_2.54mm:PinSocket_2x07_P2.54mm_Horizontal -> Glove_Footprints:PinSocket_2x07_P2.54mm_Horizontal_302-R141
Changed lines of the file:
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@@
       (effects (font (size 1.27 1.27)))
     )
-    (property "Footprint" "Connector_PinSocket_2.54mm:PinSocket_2x07_P2.54mm_Horizontal" (at 44.45 39.37 0)
+    (property "Footprint" "Glove_Footprints:PinSocket_2x07_P2.54mm_Horizontal_302-R141" (at 44.45 39.37 0)
       (effects (font (size 1.27 1.27)) hide)
     )
@@
       (effects (font (size 1.27 1.27)))
     )
-    (property "Footprint" "Connector_PinSocket_2.54mm:PinSocket_2x07_P2.54mm_Horizontal" (at 44.45 135.89 0)
-      (effects (font (size 1.27 1.27)) hide)
-    )
+    (property "Footprint" "Glove_Footprints:PinSocket_2x07_P2.54mm_Horizontal_302-R141" (at 44.45 135.89 0)
+      (effects (font (size 1.27 1.27)) hide)
+    )
