File: Hardware/glove_pcb/flex.kicad_sch (KiCad schematic)
At the start: 20 parts, among them J5 302-R141, J6 302-R141, U10 BZA408B, U11 BZA408B, U8 BZA408B, U9 BZA408B

Commit message: Changes before/after meeting w Dimitry
Connections:
- net POT_THUMB_1: now also U8.3 (K2); no longer U8.1 (K1)
- net POT_THUMB_2: now also U8.1 (K1); no longer U8.3 (K2)
Changed lines of the file:
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@@
   (junction (at 63.5 140.97) (diameter 0) (color 0 0 0 0)
   )
+  (junction (at 58.42 34.29) (diameter 0) (color 0 0 0 0)
+  )
+  (junction (at 54.61 31.75) (diameter 0) (color 0 0 0 0)
+  )
   (junction (at 147.32 72.39) (diameter 0) (color 0 0 0 0)
   )
@@
   (junction (at 33.02 143.51) (diameter 0) (color 0 0 0 0)
   )
-  (junction (at 54.61 34.29) (diameter 0) (color 0 0 0 0)
-  )
   (junction (at 96.52 138.43) (diameter 0) (color 0 0 0 0)
   )
@@
     (stroke (width 0) (type default))
   )
+  (wire (pts (xy 58.42 34.29) (xy 78.74 34.29))
+    (stroke (width 0) (type default))
+  )
   (wire (pts (xy 162.56 118.11) (xy 147.32 118.11))
     (stroke (width 0) (type default))
@@
     (stroke (width 0) (type default))
   )
-  (wire (pts (xy 54.61 34.29) (xy 78.74 34.29))
-    (stroke (width 0) (type default))
-  )
   (wire (pts (xy 33.02 36.83) (xy 36.83 36.83))
     (stroke (width 0) (type default))
@@
     (stroke (width 0) (type default))
   )
+  (wire (pts (xy 54.61 31.75) (xy 54.61 67.31))
+    (stroke (width 0) (type default))
+  )
   (wire (pts (xy 58.42 107.95) (xy 63.5 107.95))
     (stroke (width 0) (type default))
@@
     (stroke (width 0) (type default))
   )
-  (wire (pts (xy 49.53 34.29) (xy 54.61 34.29))
+  (wire (pts (xy 49.53 34.29) (xy 58.42 34.29))
     (stroke (width 0) (type default))
   )
@@
     (stroke (width 0) (type default))
   )
-  (wire (pts (xy 49.53 31.75) (xy 58.42 31.75))
+  (wire (pts (xy 49.53 31.75) (xy 54.61 31.75))
     (stroke (width 0) (type default))
   )
@@
     (stroke (width 0) (type default))
   )
+  (wire (pts (xy 54.61 31.75) (xy 58.42 31.75))
+    (stroke (width 0) (type default))
+  )
   (wire (pts (xy 87.63 64.77) (xy 87.63 72.39))
     (stroke (width 0) (type default))
@@
     (stroke (width 0) (type default))
   )
-  (wire (pts (xy 58.42 31.75) (xy 58.42 62.23))
-    (stroke (width 0) (type default))
-  )
   (wire (pts (xy 86.36 36.83) (xy 86.36 62.23))
     (stroke (width 0) (type default))
@@
     (stroke (width 0) (type default))
   )
-  (wire (pts (xy 54.61 67.31) (xy 54.61 34.29))
-    (stroke (width 0) (type default))
-  )
   (wire (pts (xy 170.18 45.72) (xy 170.18 46.99))
     (stroke (width 0) (type default))
@@
     (stroke (width 0) (type default))
   )
+  (wire (pts (xy 58.42 34.29) (xy 58.42 62.23))
+    (stroke (width 0) (type default))
+  )
