File: Hardware/glove_pcb/motor.kicad_sch (KiCad schematic)
At the start: 24 parts, among them J4 0436500200, J5 0436500200, J6 0436500200, U3 DRV8876PWPR, U4 DRV8876PWPR, U5 DRV8876PWPR

Commit message: Reworking placing
Parts:
- removed J4, J5, J6: 0436500200, Connector_JST:JST_PH_S2B-PH-K_1x02_P2.00mm_Horizontal, symbol Connector_Generic:Conn_01x02
Connections:
- net MOTOR1_OUT2: now reaches U3.10 (OUT2)
- net MOTOR1_OUT1: now reaches U3.8 (OUT1)
- net MOTOR2_OUT2: now reaches U4.10 (OUT2)
- net MOTOR2_OUT1: now reaches U4.8 (OUT1)
- net MOTOR3_OUT1: now reaches U5.8 (OUT1)
- net MOTOR3_OUT2: now reaches U5.10 (OUT2)
Other:
- note removed: "Motor"
