File: Hardware/glove_pcb/motor2.kicad_sch (KiCad schematic)
At the start: 16 parts, among them J7 0436500200, J8 0436500200, U6 DRV8876PWPR, U7 DRV8876PWPR

Commit message: Assign footprints and import all parts into pcb editor
Parts:
- J7, J8: footprint Connector_Molex:Molex_Micro-Fit_3.0_43650-0215_1x02_P3.00mm_Vertical -> Connector_Molex:Molex_Micro-Fit_3.0_43650-0200_1x02_P3.00mm_Horizontal
Changed lines of the file:
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@@
       (effects (font (size 1.27 1.27)) (justify left))
     )
-    (property "Footprint" "Connector_Molex:Molex_Micro-Fit_3.0_43650-0215_1x02_P3.00mm_Vertical" (at 248.92 48.26 0)
+    (property "Footprint" "Connector_Molex:Molex_Micro-Fit_3.0_43650-0200_1x02_P3.00mm_Horizontal" (at 248.92 48.26 0)
       (effects (font (size 1.27 1.27)) hide)
     )
@@
       (effects (font (size 1.27 1.27)) (justify left))
     )
-    (property "Footprint" "Connector_Molex:Molex_Micro-Fit_3.0_43650-0215_1x02_P3.00mm_Vertical" (at 123.19 46.99 0)
+    (property "Footprint" "Connector_Molex:Molex_Micro-Fit_3.0_43650-0200_1x02_P3.00mm_Horizontal" (at 123.19 46.99 0)
       (effects (font (size 1.27 1.27)) hide)
     )

Commit message: Re-placing with new outline
Parts:
- J7, J8: footprint Connector_Molex:Molex_Micro-Fit_3.0_43650-0200_1x02_P3.00mm_Horizontal -> Connector_JST:JST_PH_S2B-PH-K_1x02_P2.00mm_Horizontal
Changed lines of the file:
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@@
       (effects (font (size 1.27 1.27)) (justify left))
     )
-    (property "Footprint" "Connector_Molex:Molex_Micro-Fit_3.0_43650-0200_1x02_P3.00mm_Horizontal" (at 248.92 48.26 0)
+    (property "Footprint" "Connector_JST:JST_PH_S2B-PH-K_1x02_P2.00mm_Horizontal" (at 248.92 48.26 0)
       (effects (font (size 1.27 1.27)) hide)
     )
@@
       (effects (font (size 1.27 1.27)) (justify left))
     )
-    (property "Footprint" "Connector_Molex:Molex_Micro-Fit_3.0_43650-0200_1x02_P3.00mm_Horizontal" (at 123.19 46.99 0)
+    (property "Footprint" "Connector_JST:JST_PH_S2B-PH-K_1x02_P2.00mm_Horizontal" (at 123.19 46.99 0)
       (effects (font (size 1.27 1.27)) hide)
     )

Commit message: Reworking placing
Parts:
- removed J7, J8: 0436500200, Connector_JST:JST_PH_S2B-PH-K_1x02_P2.00mm_Horizontal, symbol Connector_Generic:Conn_01x02
- added J4: 0430451000, Connector_Molex:Molex_Micro-Fit_3.0_43045-1000_2x05_P3.00mm_Horizontal, symbol Connector_Generic:Conn_02x05_Top_Bottom
Connections:
- net MOTOR5_OUT1: now reaches U7.8 (OUT1)
- net MOTOR5_OUT1: now also J4.10 (Pin_10)
- net MOTOR5_OUT2: now reaches U7.10 (OUT2)
- net MOTOR5_OUT2: now also J4.5 (Pin_5)
- net MOTOR4_OUT1: now reaches U6.8 (OUT1)
- net MOTOR4_OUT1: now also J4.9 (Pin_9)
- net MOTOR4_OUT2: now reaches U6.10 (OUT2)
- net MOTOR4_OUT2: now also J4.4 (Pin_4)
- new net MOTOR1_OUT1: J4.6 (Pin_6)
- new net MOTOR1_OUT2: J4.1 (Pin_1)
- new net MOTOR2_OUT1: J4.7 (Pin_7)
- new net MOTOR2_OUT2: J4.2 (Pin_2)
- new net MOTOR3_OUT1: J4.8 (Pin_8)
- new net MOTOR3_OUT2: J4.3 (Pin_3)
Other:
- note removed: "Motor"
